File: PCB/MEISHI2022/MEISHI.kicad_sch (KiCad schematic)
At the start: 42 parts, among them IC1 TB67H450FNG,EL, IC2 TB67H450FNG,EL, J1 AC CONNECTOR, J2 USB_B_Micro, J3 AC CONNECTOR, J5 IO0, J6 IO2, J7 IO1, J8 IO3, J9 Motor Power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

Commit message: reorder files
Parts:
- removed C3: 10u, symbol Device:C_Polarized
- removed D1: POWE RLED, LED_SMD:LED_1W_3W_R8, symbol Device:LED
- removed J8: IO3, Connector_JST:JST_XH_B6B-XH-A_1x06_P2.50mm_Vertical, symbol Connector_Generic:Conn_01x06
- removed Q1: TK25S06N1L/NMOS_GDS, Package_TO_SOT_SMD:TO-252-3_TabPin2, symbol Device:Q_NMOS_GDS
- removed R2: 4.7k, Resistor_SMD:R_0603_1608Metric_Pad0.98x0.95mm_HandSolder, symbol Device:R
- removed R?: R, symbol Device:R
- added C3: 10u, Capacitor_SMD:C_0805_2012Metric_Pad1.18x1.45mm_HandSolder, symbol Device:C
- C1, C2, C4, C5, C6: footprint Capacitor_SMD:C_0603_1608Metric_Pad1.08x0.95mm_HandSolder -> Capacitor_SMD:C_0805_2012Metric_Pad1.18x1.45mm_HandSolder
- IC1, IC2: footprint Package_SO:HSOP-8-1EP_3.9x4.9mm_P1.27mm_EP2.41x3.1mm_ThermalVias -> Package_SO:HSOP-8-1EP_3.9x4.9mm_P1.27mm_EP2.41x3.1mm
- J1: value AC CONNECTOR -> AC CONNECTOR OUT
- J10, J11: renamed from J?; footprint (none) -> Connector_JST:JST_VH_B2P-VH_1x02_P3.96mm_Vertical
- J2: footprint (none) -> Project:Micro-USB-J91(Marutsu)
- J3: value AC CONNECTOR -> AC CONNECTOR IN
- J4: renamed from J?; footprint (none) -> Connector_JST:JST_XH_B4B-XH-A_1x04_P2.50mm_Vertical
- R3: renamed from R?; footprint (none) -> Resistor_SMD:R_0603_1608Metric_Pad0.98x0.95mm_HandSolder
- R6, R7: value R -> 1k
- SW1, SW2: renamed from SW?; footprint (none) -> Project:SKRPABE010
- U3: footprint RF_Module:ESP32-WROOM-32 -> Project:ESP32-WROOM-32
- gave numbers to parts that had none: 1
Connections:
- net IO3_C is gone; now on net DRIVER0_IN2: U3.10 (IO25)
- net +3V3: now also J5.2 (Pin_2), C3.2; no longer J5.1 (Pin_1)
- net +5V: now also J5.1 (Pin_1); no longer J5.2 (Pin_2)
- net DRIVER0_IN1: now also U3.9 (IO33); no longer U3.6 (IO34)
- net DRIVER0_IN2: no longer U3.9 (IO33)
- net DRIVER1_IN1: now also U3.24 (IO2); no longer U3.29 (IO5)
- net GND: now also J5.3 (Pin_3), J6.3 (Pin_3), J7.3 (Pin_3), C3.1; no longer J5.6 (Pin_6), J6.6 (Pin_6), J7.6 (Pin_6)
- net IO0_A: now also J5.4 (Pin_4), U3.13 (IO14); no longer J5.3 (Pin_3), U3.14 (IO12)
- net IO0_B: now also J5.5 (Pin_5), U3.14 (IO12); no longer J5.4 (Pin_4), U3.16 (IO13)
- net IO0_C: now also J5.6 (Pin_6), U3.16 (IO13); no longer J5.5 (Pin_5), U3.13 (IO14)
- net IO1_A: now also J7.4 (Pin_4); no longer J7.3 (Pin_3)
- net IO1_B: now also J7.5 (Pin_5); no longer J7.4 (Pin_4)
- net IO1_C: now also J7.6 (Pin_6); no longer J7.5 (Pin_5)
- net IO2_A: now also J6.4 (Pin_4); no longer J6.3 (Pin_3)
- net IO2_B: now also J6.5 (Pin_5); no longer J6.4 (Pin_4)
- net IO2_C: now also J6.6 (Pin_6); no longer J6.5 (Pin_5)
- net at J3.2 (Pin_2): now also K1.5 (NO_2); no longer K1.3 (COM_1)
- net AC_OUT2: now reaches J1.1 (Pin_1)
- net AC_OUT2: now also K1.6 (COM_2), K1.7 (NC_2); no longer K1.5 (NO_2)
- net AC_OUT1: now reaches J1.2 (Pin_2)
- net AC_OUT1: now also K1.2 (NC_1), K1.3 (COM_1); no longer K1.6 (COM_2)
- net IO3_A: no longer names the net of U3.36 (IO22)
- net IO3_B: no longer names the net of U3.37 (IO23)
- net POWER LED: no longer names the net of U3.8 (IO32)
- no-connect marks 15 -> 17
Other:
- note added: "2.54mm IO IO0 , IO1 5 3.3 G A B C IO2 , IO3 3.3 5 G A B C"
- note removed: "2.54mm IO 3.3 5 G A B C"
- note removed: "Power LED"
- moved on the sheet: J1, J10, J11, J3

Commit message: feat MEISHI
Parts:
- J10, J11: footprint Connector_JST:JST_VH_B2P-VH_1x02_P3.96mm_Vertical -> Connector_JST:JST_XA_B02B-XASK-1_1x02_P2.50mm_Vertical
Changed lines of the file:
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@@
       (effects (font (size 1.27 1.27)) (justify left))
     )
-    (property "Footprint" "Connector_JST:JST_VH_B2P-VH_1x02_P3.96mm_Vertical" (id 2) (at 207.518 150.876 0)
+    (property "Footprint" "Connector_JST:JST_XA_B02B-XASK-1_1x02_P2.50mm_Vertical" (id 2) (at 207.518 150.876 0)
       (effects (font (size 1.27 1.27)) hide)
     )
@@
       (effects (font (size 1.27 1.27)) (justify left))
     )
-    (property "Footprint" "Connector_JST:JST_VH_B2P-VH_1x02_P3.96mm_Vertical" (id 2) (at 207.518 141.732 0)
+    (property "Footprint" "Connector_JST:JST_XA_B02B-XASK-1_1x02_P2.50mm_Vertical" (id 2) (at 207.518 141.732 0)
       (effects (font (size 1.27 1.27)) hide)
     )
@@
     )
     (path "/69b192a7-07ce-41c4-aecc-def9ea6cfe05"
-      (reference "J10") (unit 1) (value "Motor0") (footprint "Connector_JST:JST_VH_B2P-VH_1x02_P3.96mm_Vertical")
+      (reference "J10") (unit 1) (value "Motor0") (footprint "Connector_JST:JST_XA_B02B-XASK-1_1x02_P2.50mm_Vertical")
     )
     (path "/3731bcf0-c6cc-4b6e-b21e-15049107b33f"
-      (reference "J11") (unit 1) (value "Motor1") (footprint "Connector_JST:JST_VH_B2P-VH_1x02_P3.96mm_Vertical")
+      (reference "J11") (unit 1) (value "Motor1") (footprint "Connector_JST:JST_XA_B02B-XASK-1_1x02_P2.50mm_Vertical")
     )
     (path "/e14349e4-a419-4f53-a4c3-d5fab413fc98"

Commit message: fix pcb
Parts:
- removed J9: Motor Power, Connector_JST:JST_VH_B2P-VH_1x02_P3.96mm_Vertical, symbol Connector_Generic:Conn_01x02
- added J8: Motor Power, Connector_JST:JST_XA_B03B-XASK-1_1x03_P2.50mm_Vertical, symbol Connector_Generic:Conn_01x03
Connections:
- net +5V: now also K1.1 (COIL_1); no longer K1.8 (COIL_2)
- net GND: now also J8.3 (Pin_3)
- net VCC: now also J8.1 (Pin_1)
- net at D2.2 (A), U2.6: now also K1.8 (COIL_2); no longer K1.1 (COIL_1)
- no-connect marks 17 -> 20
Other:
- moved on the sheet: D2, J1, J3, K1
