File: PCB/MEISHI2022/MEISHI.kicad_pcb (KiCad board)
At the start: 2 copper layers, 91 x 55 mm, 0 parts

Commit message: reorder files
Parts:
- added C1: 10u, Capacitor_SMD:C_0805_2012Metric_Pad1.18x1.45mm_HandSolder, F.Cu at (29.7, 67.2)
- added C2: 22u, Capacitor_SMD:C_0805_2012Metric_Pad1.18x1.45mm_HandSolder, F.Cu at (33.6, 63.2)
- added C3: 10u, Capacitor_SMD:C_0805_2012Metric_Pad1.18x1.45mm_HandSolder, F.Cu at (33.6, 61.2)
- added C4: 0.1u, Capacitor_SMD:C_0805_2012Metric_Pad1.18x1.45mm_HandSolder, F.Cu at (33.6, 59.1)
- added C5: 0.1u, Capacitor_SMD:C_0805_2012Metric_Pad1.18x1.45mm_HandSolder, F.Cu at (87.2, 38.8)
- added C6: 0.1u, Capacitor_SMD:C_0805_2012Metric_Pad1.18x1.45mm_HandSolder, F.Cu at (65.6, 66.6)
- added D2: D, Diode_SMD:D_SOD-128, F.Cu at (74.0, 51.8)
- added IC1: TB67H450FNG,EL, Package_SO:HSOP-8-1EP_3.9x4.9mm_P1.27mm_EP2.41x3.1mm, F.Cu at (61.8, 61.3)
- added IC2: TB67H450FNG,EL, Package_SO:HSOP-8-1EP_3.9x4.9mm_P1.27mm_EP2.41x3.1mm, F.Cu at (87.2, 34.8)
- added J1: AC CONNECTOR OUT, Connector_JST:JST_VH_B2P-VH_1x02_P3.96mm_Vertical, F.Cu at (93.8, 71.8)
- added J10: Motor0, Connector_JST:JST_VH_B2P-VH_1x02_P3.96mm_Vertical, F.Cu at (69.8, 69.2)
- added J11: Motor1, Connector_JST:JST_VH_B2P-VH_1x02_P3.96mm_Vertical, F.Cu at (102.7, 29.2)
- added J2: USB_B_Micro, Project:Micro-USB-J91(Marutsu), F.Cu at (25.4, 72.9)
- added J3: AC CONNECTOR IN, Connector_JST:JST_VH_B2P-VH_1x02_P3.96mm_Vertical, F.Cu at (103.7, 71.8)
- added J4: Conn_01x04, Connector_JST:JST_XH_B4B-XH-A_1x04_P2.50mm_Vertical, F.Cu at (43.6, 25.5)
- added J5: IO0, Connector_JST:JST_XH_B6B-XH-A_1x06_P2.50mm_Vertical, F.Cu at (44.2, 69.4)
- added J6: IO2, Connector_JST:JST_XH_B6B-XH-A_1x06_P2.50mm_Vertical, F.Cu at (62.9, 25.5)
- added J7: IO1, Connector_JST:JST_XH_B6B-XH-A_1x06_P2.50mm_Vertical, F.Cu at (87.5, 25.5)
- added J9: Motor Power, Connector_JST:JST_VH_B2P-VH_1x02_P3.96mm_Vertical, F.Cu at (102.2, 45.0)
- added K1: 942H-2C-5DS, Project:942H2C5DS, F.Cu at (80.0, 59.8)
- added LS1: Speaker_Ultrasound, Buzzer_Beeper:Buzzer_TDK_PS1240P02BT_D12.2mm_H6.5mm, F.Cu at (70.8, 34.6)
- added R1: 1k, Resistor_SMD:R_0603_1608Metric_Pad0.98x0.95mm_HandSolder, F.Cu at (68.9, 48.4)
- added R10: 0.1, Resistor_SMD:R_1210_3225Metric_Pad1.30x2.65mm_HandSolder, F.Cu at (82.7, 30.4)
- added R11: 0.1, Resistor_SMD:R_1210_3225Metric_Pad1.30x2.65mm_HandSolder, F.Cu at (63.6, 55.0)
- added R13: 4.7k, Resistor_SMD:R_0603_1608Metric_Pad0.98x0.95mm_HandSolder, F.Cu at (30.9, 27.0)
- added R3: R, Resistor_SMD:R_0603_1608Metric_Pad0.98x0.95mm_HandSolder, F.Cu at (73.3, 45.6)
- added R4: 110, Resistor_SMD:R_0603_1608Metric_Pad0.98x0.95mm_HandSolder, F.Cu at (46.8, 61.0)
- added R5: 4.7k, Resistor_SMD:R_0603_1608Metric_Pad0.98x0.95mm_HandSolder, F.Cu at (42.2, 65.2)
- added R6: 1k, Resistor_SMD:R_0603_1608Metric_Pad0.98x0.95mm_HandSolder, F.Cu at (79.0, 44.0)
- added R7: 1k, Resistor_SMD:R_0603_1608Metric_Pad0.98x0.95mm_HandSolder, F.Cu at (79.0, 45.6)
- added R8: 1k, Resistor_SMD:R_0603_1608Metric_Pad0.98x0.95mm_HandSolder, F.Cu at (59.2, 65.5)
- added R9: 1k, Resistor_SMD:R_0603_1608Metric_Pad0.98x0.95mm_HandSolder, F.Cu at (62.6, 65.5)
- added SW1: SW_MEC_5E, Project:SKRPABE010, F.Cu at (41.2, 61.4)
- added SW2: SW_MEC_5E, Project:SKRPABE010, F.Cu at (25.0, 25.0)
- added U1: AZ1117-3.3, Package_TO_SOT_SMD:SOT-223-3_TabPin2, F.Cu at (36.1, 68.4)
- added U2: TLP172AM, Package_SO:MFSOP6-4_4.4x3.6mm_P1.27mm, F.Cu at (70.8, 57.4)
- added U3: ESP32-WROOM-32D, Project:ESP32-WROOM-32, F.Cu at (41.2, 47.3)
Routing:
- net +3V3: track 0.00 -> 176.6 mm, vias 0 -> 2
- net +5V: track 0.00 -> 152.4 mm, vias 0 -> 1
- net VCC: track 0.00 -> 66.0 mm, vias 0 -> 2
- net GND: track 0.00 -> 52.4 mm, vias 0 -> 25
- net /DRIVER1_IN2: track 0.00 -> 39.6 mm, vias 0 -> 2
- net /IO1_A: track 0.00 -> 39.1 mm
- net Net-(R13-Pad2): track 0.00 -> 37.6 mm, vias 0 -> 2
- net /IO1_B: track 0.00 -> 36.6 mm
- net /IO1_C: track 0.00 -> 36.3 mm
- net /DRIVER1_IN1: track 0.00 -> 34.3 mm, vias 0 -> 2
- net /BUSSER: track 0.00 -> 32.4 mm, vias 0 -> 2
- net /AC_OUT2: track 0.00 -> 31.2 mm
- net Net-(R4-Pad1): track 0.00 -> 29.0 mm, vias 0 -> 2
- net /DRIVER0_IN1: track 0.00 -> 27.3 mm, vias 0 -> 2
- net /DRIVER0_IN2: track 0.00 -> 24.7 mm, vias 0 -> 2
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- added copper zone on B.Cu, net GND
- added copper zone on F.Cu, net GND

Commit message: feat MEISHI
Parts:
- J10, J11: footprint Connector_JST:JST_VH_B2P-VH_1x02_P3.96mm_Vertical -> Connector_JST:JST_XA_B02B-XASK-1_1x02_P2.50mm_Vertical
- moved SW2 94.2 mm to (106.5, 72.4), turned to 0 degrees
- moved J2 94.0 mm to (106.1, 24.5), turned to 180 degrees
- moved J3 88.8 mm to (27.8, 25.6), turned to -90 degrees
- moved J11 83.5 mm to (28.8, 68.2), turned to -90 degrees
- moved R13 82.1 mm to (100.5, 70.4), turned to 0 degrees
- moved C1 80.9 mm to (101.7, 30.2), turned to 0 degrees
- moved J9 73.3 mm to (29.3, 52.4), turned to -90 degrees
- moved J1 72.7 mm to (37.7, 25.6), turned to -90 degrees
- moved U1 71.1 mm to (95.3, 29.0), turned to 180 degrees
- moved C2 70.5 mm to (97.9, 34.1), turned to 0 degrees
- moved C3 69.0 mm to (97.9, 36.2), turned to 180 degrees
- moved C4 67.5 mm to (97.9, 38.3), turned to 180 degrees
- moved J4 64.1 mm to (87.9, 71.9), turned to 0 degrees
- moved J7 63.5 mm to (44.0, 71.9), turned to 0 degrees
- moved J5 59.6 mm to (87.2, 28.0), turned to 180 degrees
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Routing:
- net GND: track 52.4 -> 56.7 mm, vias 25 -> 91
- net Net-(LS1-Pad1): track 20.2 -> 18.8 mm
- net /DRIVER1_OUT2: track 15.8 -> 15.2 mm
- net (no net): vias 1 -> 0
Other:
- board text added: "3.3"
- board text added: "5"
- board text added: "5V"
- board text added: "A0"
- board text added: "A1"
- board text added: "A2"
- board text added: "AC 100V"
- board text added: "AC IN"
- board text added: "AC OUT"
- board text added: "B0"
- board text added: "B1"
- board text added: "B2"
- board text added: "C0"
- board text added: "C1"
- board text added: "C2"
- board text added: "DANGER ZONE"
- board text added: "G"
- board text added: "GND"
- board text added: "HIGH VOLTAGE"
- board text added: "Motor Power"
- board text added: "Motor0"
- board text added: "Motor1"
- board text added: "RX0"
- board text added: "TX0"

Commit message: fix pcb
Parts:
- removed J9: Motor Power, Connector_JST:JST_VH_B2P-VH_1x02_P3.96mm_Vertical
- added J8: Motor Power, Connector_JST:JST_XA_B03B-XASK-1_1x03_P2.50mm_Vertical, F.Cu at (29.2, 52.5)
- moved SW2 37.6 mm to (76.2, 50.0), turned to 90 degrees
- moved R13 25.9 mm to (77.2, 59.2)
- moved D2 16.3 mm to (50.4, 30.9), turned to 180 degrees
- moved R10 12.4 mm to (36.4, 65.7), turned to 180 degrees
- moved R3 10.7 mm to (68.1, 47.8), turned to 180 degrees
- moved R1 9.14 mm to (71.6, 47.8)
- moved R6 8.91 mm to (49.3, 61.7), turned to 90 degrees
- moved R7 7.12 mm to (49.3, 58.2), turned to 90 degrees
- moved U2 7.10 mm to (59.4, 47.0)
- moved LS1 5.42 mm to (63.0, 57.9), turned to -90 degrees
- moved J11 3.81 mm to (29.2, 64.5)
- moved C1 1.12 mm to (101.0, 31.1), turned to -90 degrees
Connections:
- K1 pad 1: Net-(D2-Pad2) -> +5V
- K1 pad 8: +5V -> Net-(D2-Pad2)
Routing:
- net Net-(R13-Pad2): track 37.6 -> 13.8 mm
- net +5V: track 152.4 -> 173.4 mm
- net GND: track 56.7 -> 41.2 mm, vias 91 -> 93
- net Net-(D2-Pad2): track 9.72 -> 21.7 mm
- net /BUSSER: track 32.4 -> 21.9 mm
- net VCC: track 66.0 -> 74.4 mm, vias 2 -> 4
- net Net-(IC2-Pad4): track 11.2 -> 4.14 mm
- net Net-(IC2-Pad7): track 9.98 -> 4.67 mm, vias 2 -> 0
- net Net-(LS1-Pad1): track 18.8 -> 15.7 mm
- net /DRIVER1_IN1: track 34.3 -> 36.6 mm
- net /IO1_A: track 39.1 -> 37.0 mm
- net /DRIVER1_OUT1: track 15.3 -> 13.5 mm
- net +3V3: track 176.6 -> 178.3 mm
- net /DRIVER1_IN2: track 39.6 -> 38.4 mm
- net Net-(J3-Pad1): track 16.7 -> 17.8 mm
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Other:
- outline, holes or cut-outs redrawn
- board text added: "+"
- board text added: "CAUTION HV"
- board text added: "MEISHI v1.0"
- board text removed: "DANGER ZONE"
- board text removed: "HIGH VOLTAGE"

Commit message: update
Parts:
- renumbered J8 to Je
Changed lines of the file:
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@@
     (property "Sheetname" "")
     (attr through_hole)
-    (fp_text reference "J8" (at 2.5 -4.4 -90) (layer "F.SilkS")
+    (fp_text reference "Je" (at 2.5 -4.4 -90) (layer "F.SilkS") hide
       (effects (font (size 1 1) (thickness 0.15)))
     )
